Commit message: Update finger.urdf

File: isaacgym/finger.urdf (robot description, URDF)
Before this commit: robot conveyor, 1 links, 0 joints
Links:
- link baseLink: geometry collision mesh filename=/home/tasha/PycharmProjects/robotics/assets/meshes/collisio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; visual mesh filename=/home/tasha/PycharmProjects/robotics/assets/meshes/visual/s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
